File: _autosave-Power.kicad_sch (KiCad schematic)
At the start: 0 parts

Commit message: using ultra lib symbols instead of custom and adding to sym table
Parts:
- added C? (x7): 10muF, symbol Device:C_Small
- added C? (x5): 0.1muF, symbol Device:C_Small
- added C?: 1muF, symbol Device:C_Small
- added C?: 47muF, symbol Device:C_Small
- added L?: 1uH, symbol Device:L
- added R?: 10K, symbol Device:R_Small_US
- added R? (x2): 4.4k, symbol Device:R_Small_US
- added R? (x2): 3.3k, symbol Device:R_Small_US
- added R?: 10k, symbol Device:R_Small_US
- added R?: 100k, symbol Device:R_Small_US
- added U?: LMS36353QRNLRQ1, RNL0022A, symbol LMS3635-Q1:LMS36353QRNLRQ1
- added U?: LP87702DRHBRQ1, RHB0032N, symbol LP87702DRHBRQ1:LP87702DRHBRQ1
- added U?: PTPS7A5310AQWRTJQ1, WQFN20_RTJ_TEX, symbol TPS7A5301QRGRRQ1:PTPS7A5310AQWRTJQ1
Connections:
- new net: R?.2, U?.1 (INT_N)
- new net: L?.1, U?.9 (SW_BST)
- new net: C?.2, U?.13 (NR/SS)
- new net +1V35: C?.1, C?.1, C?.1, C?.1, C?.1, C?.1, C?.2, C?.2, C?.2, C?.2, C?.2, C?.2, R?.2, U?.14 (EN), U?.15 (IN), U?.16 (IN), U?.17 (IN), U?.17 (PGND_B1), U?.18 (PGND_B1), U?.22 (CLKIN_GPO2), U?.23 (PGND_B0), U?.24 (PGND_B0)
- new net +3V3: C?.1, C?.1, C?.1, C?.2, C?.2, L?.2, R?.1, R?.1, R?.1, R?.1, U?.12 (BIAS), U?.13 (VIN_B1), U?.14 (VIN_B1), U?.27 (VIN_B0), U?.28 (VIN_B0)
- new net AWR_SCL: R?.2, U?.20 (SCL_EN2)
- new net AWR_SDA: R?.2, U?.21 (SDA_EN3)
- new net PMIC_EN1: U?.11 (NRST), U?.19 (EN1)
- new net TP2: U?.4 (PG)
- new net VCC_LDO_OUT: C?.1, C?.1, C?.1, C?.2, C?.2, C?.2, U?.1 (OUT), U?.19 (OUT), U?.20 (OUT)
