File: _autosave-stm32h7_core.kicad_sch (KiCad schematic)
At the start: 22 parts, among them SW2 RST_BTN, U3 STM32H743ZITx

Commit message: squasing ERC errors
Parts:
- removed C10, C11, C12, C13, C14, C15, C16, C17, C18, C19, C5, C6, C7, C8, C9: 100nF, symbol Device:C_Small
- removed C20: 100nf, symbol Device:C_Small
- removed D1: D_TVS, symbol Device:D_TVS
- removed FB1: ?, symbol Device:FerriteBead
- removed R10, R11: 10K, symbol Device:R_Small_US
- removed SW2: RST_BTN, symbol Switch:SW_DIP_x01
- removed U3: STM32H743ZITx, Package_QFP:LQFP-144_20x20mm_P0.5mm, symbol MCU_ST_STM32H7:STM32H743ZITx
