File: _autosave-awr1843.kicad_sch (KiCad schematic)
At the start: 0 parts

Commit message: making unit design for AWR1843, starting with GND, voltage, I2C and GPIO
Other:
- added sheet awr_pwrpins (awr_pwr.kicad_sch)
Changed lines of the file:
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@@
 (kicad_sch (version 20230121) (generator eeschema)
   (paper "A4")
+  (sheet (at 31.75 27.94) (size 48.26 30.48) (fields_autoplaced)
+    (stroke (width 0.1524) (type solid))
+    (fill (color 0 0 0 0.0000))
+    (property "Sheetname" "awr_pwrpins" (at 31.75 27.2284 0)
+      (effects (font (size 1.27 1.27)) (justify left bottom))
+    )
+    (property "Sheetfile" "awr_pwr.kicad_sch" (at 31.75 59.0046 0)
+      (effects (font (size 1.27 1.27)) (justify left top))
+    )
+    (instances
+      (project "radar"
+        (path "/88b309aa-5f0e-45d7-beec-81d4b0ee2121/a7a83c3c-ff2f-4f3c-a80e-562a1762ef83" (page "6"))
+      )
+    )
+  )
 )
