File: 16flashmem.kicad_sch (KiCad schematic)
At the start: 0 parts

Commit message: finishing flash schematic
Parts:
- added C8: 1muF, symbol Device:C_Small
- added C9: 0.1muF, symbol Device:C_Small
- added IC1: MX25V1635FZNQ03-T, SON127P600X500X80-9N-D, symbol MX25V1635FZNQ03-T:MX25V1635FZNQ03-T
- added R30, R31, R32: 10k, symbol Device:R_Small_US
- added R33, R34, R35: 33.2k, symbol Device:R_Small_US
Connections:
- new net: IC1.2 (SO/SIO1), R33.1
- new net: IC1.5 (SI/SIO0), R35.2
- new net: IC1.6 (SCLK), R34.2
- new net +3V3: C8.1, C8.2, C9.1, C9.2, IC1.4 (GND), IC1.8 (VCC), IC1.9 (EP), R30.1, R31.1, R32.1
- new net AWR_QSPI_CLK: R34.1
- new net AWR_QSPI_CS: IC1.1 (CS#), R30.2
- new net AWR_QSPI_D0: R35.1
- new net AWR_QSPI_D1: R33.2
- new net AWR_QSPI_D2: IC1.3 (WP#/SIO2), R32.2
- new net AWR_QSPI_D3: IC1.7 (HOLD#/SIO3), R31.2

Commit message: decoup and lc schematics
Other:
- moved on the sheet: C8, C9, IC1, R30, R31, R32, R33, R34, R35
