File: 16flashmem.kicad_sch (KiCad schematic)
At the start: 9 parts, among them IC1 MX25V1635FZNQ03-T

Commit message: adding footprints
Parts:
- C8, C9: footprint (none) -> Capacitor_SMD:C_0603_1608Metric
- IC1: footprint SON127P600X500X80-9N-D -> MX25:SON127P600X500X80-9N-D
- R30, R31, R32, R33, R34, R35: footprint (none) -> Resistor_SMD:R_0603_1608Metric
Changed lines of the file:
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@@
       (effects (font (size 1.27 1.27)))
     )
-    (property "Footprint" "SON127P600X500X80-9N-D" (at 146.05 190.17 0)
+    (property "Footprint" "MX25:SON127P600X500X80-9N-D" (at 146.05 190.17 0)
       (effects (font (size 1.27 1.27)) (justify left top) hide)
     )
@@
       (effects (font (size 1.27 1.27)))
     )
-    (property "Footprint" "" (at 99.06 97.79 0)
+    (property "Footprint" "Resistor_SMD:R_0603_1608Metric" (at 99.06 97.79 0)
       (effects (font (size 1.27 1.27)) hide)
     )
@@
       (effects (font (size 1.27 1.27)) (justify left))
     )
-    (property "Footprint" "" (at 176.53 80.01 0)
+    (property "Footprint" "Capacitor_SMD:C_0603_1608Metric" (at 176.53 80.01 0)
       (effects (font (size 1.27 1.27)) hide)
     )
@@
       (effects (font (size 1.27 1.27)) (justify left))
     )
-    (property "Footprint" "" (at 95.25 73.66 0)
+    (property "Footprint" "Resistor_SMD:R_0603_1608Metric" (at 95.25 73.66 0)
       (effects (font (size 1.27 1.27)) hide)
     )
@@
       (effects (font (size 1.27 1.27)) (justify left))
     )
-    (property "Footprint" "" (at 59.69 106.68 0)
+    (property "Footprint" "Resistor_SMD:R_0603_1608Metric" (at 59.69 106.68 0)
       (effects (font (size 1.27 1.27)) hide)
     )
@@
       (effects (font (size 1.27 1.27)) (justify left))
     )
-    (property "Footprint" "" (at 208.28 92.71 0)
+    (property "Footprint" "Resistor_SMD:R_0603_1608Metric" (at 208.28 92.71 0)
       (effects (font (size 1.27 1.27)) hide)
     )
@@
       (effects (font (size 1.27 1.27)))
     )
-    (property "Footprint" "" (at 161.29 130.81 0)
+    (property "Footprint" "Resistor_SMD:R_0603_1608Metric" (at 161.29 130.81 0)
       (effects (font (size 1.27 1.27)) hide)
     )
@@
       (effects (font (size 1.27 1.27)))
     )
-    (property "Footprint" "" (at 167.64 120.65 0)
+    (property "Footprint" "Resistor_SMD:R_0603_1608Metric" (at 167.64 120.65 0)
       (effects (font (size 1.27 1.27)) hide)
     )
@@
       (effects (font (size 1.27 1.27)) (justify left))
     )
-    (property "Footprint" "" (at 160.02 80.01 0)
-      (effects (font (size 1.27 1.27)) hide)
-    )
+    (property "Footprint" "Capacitor_SMD:C_0603_1608Metric" (at 160.02 80.01 0)
+      (effects (font (size 1.27 1.27)) hide)
+    )
