File: Power.kicad_sch (KiCad schematic)
At the start: 34 parts, among them U1 LP87702DRHBRQ1

Commit message: decoup and lc schematics
Connections:
- net AWR_1V2 is gone; now on net 1V24: R8.2
- net AWR_1V8 is gone; now on net 1V8: R9.2
- net 1V2 renamed 1V24
Other:
- added sheet decoup_caps (decoup_caps.kicad_sch)
- added sheet lc_filter (lc_filter.kicad_sch)
Changed lines of the file:
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@@
     (stroke (width 0) (type default))
   )
-  (wire (pts (xy 170.18 62.23) (xy 170.18 66.04))
+  (wire (pts (xy 173.99 64.77) (xy 173.99 66.04))
     (stroke (width 0) (type default))
   )
@@
     (stroke (width 0) (type default))
   )
+  (wire (pts (xy 170.18 64.77) (xy 170.18 62.23))
+    (stroke (width 0) (type default))
+  )
   (wire (pts (xy 48.26 101.6) (xy 41.91 101.6))
     (stroke (width 0) (type default))
@@
   )
   (wire (pts (xy 29.21 63.5) (xy 29.21 71.12))
+    (stroke (width 0) (type default))
+  )
+  (wire (pts (xy 173.99 64.77) (xy 170.18 64.77))
     (stroke (width 0) (type default))
   )
@@
     )
   )
-  (global_label "AWR_1V2" (shape input) (at 101.6 168.91 0) (fields_autoplaced)
+  (global_label "1V24" (shape input) (at 101.6 168.91 0) (fields_autoplaced)
     (effects (font (size 1.27 1.27)) (justify left))
-    (property "Intersheetrefs" "${INTERSHEET_REFS}" (at 112.8704 168.91 0)
+    (property "Intersheetrefs" "${INTERSHEET_REFS}" (at 109.3023 168.91 0)
       (effects (font (size 1.27 1.27)) (justify left) hide)
     )
@@
     )
   )
-  (global_label "AWR_1V8" (shape input) (at 125.73 129.54 0) (fields_autoplaced)
+  (global_label "1V8" (shape input) (at 125.73 129.54 0) (fields_autoplaced)
     (effects (font (size 1.27 1.27)) (justify left))
-    (property "Intersheetrefs" "${INTERSHEET_REFS}" (at 137.0004 129.54 0)
+    (property "Intersheetrefs" "${INTERSHEET_REFS}" (at 132.2228 129.54 0)
       (effects (font (size 1.27 1.27)) (justify left) hide)
     )
@@
     )
   )
-  (global_label "1V2" (shape input) (at 158.75 68.58 0) (fields_autoplaced)
+  (global_label "1V24" (shape input) (at 158.75 68.58 0) (fields_autoplaced)
     (effects (font (size 1.27 1.27)) (justify left))
-    (property "Intersheetrefs" "${INTERSHEET_REFS}" (at 165.2428 68.58 0)
+    (property "Intersheetrefs" "${INTERSHEET_REFS}" (at 166.4523 68.58 0)
       (effects (font (size 1.27 1.27)) (justify left) hide)
     )
@@
     )
   )
-  (symbol (lib_id "power:GND") (at 170.18 66.04 0) (unit 1)
-    (in_bom yes) (on_board yes) (dnp no) (fields_autoplaced)
-    (property "Reference" "#PWR024" (at 170.18 72.39 0)
-      (effects (font (size 1.27 1.27)) hide)
-    )
-    (property "Value" "GND" (at 170.18 71.12 0)
-      (effects (font (size 1.27 1.27)))
-    )
-    (property "Footprint" "" (at 170.18 66.04 0)
-      (effects (font (size 1.27 1.27)) hide)
-    )
-    (property "Datasheet" "" (at 170.18 66.04 0)
+  (symbol (lib_id "power:GND") (at 173.99 66.04 0) (unit 1)
+    (in_bom yes) (on_board yes) (dnp no) (fields_autoplaced)
+    (property "Reference" "#PWR024" (at 173.99 72.39 0)
+      (effects (font (size 1.27 1.27)) hide)
+    )
+    (property "Value" "GND" (at 173.99 71.12 0)
+      (effects (font (size 1.27 1.27)))
+    )
+    (property "Footprint" "" (at 173.99 66.04 0)
+      (effects (font (size 1.27 1.27)) hide)
+    )
+    (property "Datasheet" "" (at 173.99 66.04 0)
       (effects (font (size 1.27 1.27)) hide)
     )
@@
     )
   )
-  (sheet (at 220.98 20.32) (size 57.15 139.7) (fields_autoplaced)
+  (sheet (at 220.98 95.25) (size 55.88 16.51) (fields_autoplaced)
+    (stroke (width 0.1524) (type solid))
+    (fill (color 0 0 0 0.0000))
+    (property "Sheetname" "decoup_caps" (at 220.98 94.5384 0)
+      (effects (font (size 1.27 1.27)) (justify left bottom))
+    )
+    (property "Sheetfile" "decoup_caps.kicad_sch" (at 220.98 112.3446 0)
+      (effects (font (size 1.27 1.27)) (justify left top))
+    )
+    (property "Field2" "" (at 220.98 95.25 0)
+      (effects (font (size 1.27 1.27)) hide)
+    )
+    (instances
+      (project "radar"
+        (path "/88b309aa-5f0e-45d7-beec-81d4b0ee2121/7a3c78f1-80f2-463b-a37f-9a7b3cc7f964" (page "8"))
+      )
+    )
+  )
+  (sheet (at 220.98 68.58) (size 57.15 13.97) (fields_autoplaced)
+    (stroke (width 0.1524) (type solid))
+    (fill (color 0 0 0 0.0000))
+    (property "Sheetname" "lc_filter" (at 220.98 67.8684 0)
+      (effects (font (size 1.27 1.27)) (justify left bottom))
+    )
+    (property "Sheetfile" "lc_filter.kicad_sch" (at 220.98 83.1346 0)
+      (effects (font (size 1.27 1.27)) (justify left top))
+    )
+    (instances
+      (project "radar"
+        (path "/88b309aa-5f0e-45d7-beec-81d4b0ee2121/7a3c78f1-80f2-463b-a37f-9a7b3cc7f964" (page "7"))
+      )
+    )
+  )
+  (sheet (at 220.98 20.32) (size 58.42 35.56) (fields_autoplaced)
     (stroke (width 0.1524) (type solid))
     (fill (color 0 0 0 0.0000))
@@
       (effects (font (size 1.27 1.27)) (justify left bottom))
     )
-    (property "Sheetfile" "stepdwn_and_ldo.kicad_sch" (at 220.98 160.6046 0)
+    (property "Sheetfile" "stepdwn_and_ldo.kicad_sch" (at 220.98 56.4646 0)
       (effects (font (size 1.27 1.27)) (justify left top))
     )
