File: awr1843.kicad_sch (KiCad schematic)
At the start: 0 parts

Commit message: decoup and lc schematics
Parts:
- added U3, U6: AWR1843ABG_, symbol AWR1843ABGABLRQ1:AWR1843ABG_
Connections:
- new net AWR_1V0_RF1: U3.G5 (VIN_13RF1), U3.H5 (VIN_13RF1), U3.J5 (VIN_13RF1)
- new net AWR_1V0_RF2: U3.C2 (VIN_13RF2), U3.D2 (VIN_13RF2)
- new net AWR_1V24: U3.G15 (VIN_SRAM), U3.N11 (VDDIN), U3.P14 (VNWA), U3.P15 (VDDIN), U3.R6 (VDDIN)
- new net AWR_1V8: U3.B11 (VIN_18CLK), U3.B12 (VIN_18VCO), U3.D15 (VIOIN_18DIFF), U3.K5 (VIN_18BB), U3.R9 (VIOIN_18)
- new net AWR_3V3: U3.F15 (VIOIN), U3.R10 (VIOIN)
- new net GND: U3.A1 (VSSA), U3.A13 (VSSA), U3.A15 (VSSA), U3.A3 (VSSA), U3.A5 (VSSA), U3.A7 (VSSA), U3.A9 (VSSA), U3.B1 (VSSA), U3.B14 (VSSA), U3.B3 (VSSA), U3.B5 (VSSA), U3.B7 (VSSA), U3.B9 (VSSA), U3.C1 (VSSA), U3.C14 (VSSA), U3.C3 (VSSA), U3.C4 (VSSA), U3.C5 (VSSA), U3.C6 (VSSA), U3.C7 (VSSA), U3.C8 (VSSA), U3.C9 (VSSA), U3.E1 (VSSA), U3.E10 (VSS), U3.E2 (VSSA), U3.E3 (VSSA), U3.E5 (VSS), U3.E6 (VSS), U3.E8 (VSS), U3.F11 (VSS), U3.F3 (VSSA), U3.F9 (VSS), U3.G1 (VSSA), U3.G10 (VSS), U3.G2 (VSSA), U3.G3 (VSSA), U3.G6 (VSS), U3.G7 (VSS), U3.G8 (VSS), U3.H11 (VSS), U3.H3 (VSSA), U3.H7 (VSS), U3.H9 (VSS), U3.J1 (VSSA), U3.J10 (VSS), U3.J2 (VSSA), U3.J3 (VSSA), U3.J6 (VSS), U3.J7 (VSS), U3.J8 (VSS), U3.K10 (VSS), U3.K11 (VSS), U3.K3 (VSSA), U3.K7 (VSS), U3.K8 (VSS), U3.K9 (VSS), U3.L1 (VSSA), U3.L10 (VSS), U3.L2 (VSSA), U3.L3 (VSSA), U3.L5 (VSS), U3.L6 (VSS), U3.L8 (VSS), U3.M3 (VSSA), U3.N1 (VSSA), U3.N2 (VSSA), U3.N3 (VSSA), U3.R1 (VSSA), U3.R15 (VSS)
