File: stepdwn_and_ldo.kicad_sch (KiCad schematic)
At the start: 48 parts, among them J1 USB_C_Receptacle_USB2.0_14P, U2 BQ25895RTW, U4 PTPS7A5310AQWRTJQ1, U5 LMS36353QRNLRQ1

Commit message: decoup and lc schematics
Connections:
- net AVIN (LMS) renamed +5V
Changed lines of the file:
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@@
   (junction (at 231.14 72.39) (diameter 0) (color 0 0 0 0)
+  )
+  (junction (at 252.73 53.34) (diameter 0) (color 0 0 0 0)
   )
   (junction (at 243.84 53.34) (diameter 0) (color 0 0 0 0)
@@
     (stroke (width 0) (type default))
   )
-  (wire (pts (xy 243.84 53.34) (xy 261.62 53.34))
+  (wire (pts (xy 243.84 53.34) (xy 252.73 53.34))
     (stroke (width 0) (type default))
   )
@@
     (stroke (width 0) (type default))
   )
+  (wire (pts (xy 252.73 53.34) (xy 261.62 53.34))
+    (stroke (width 0) (type default))
+  )
   (wire (pts (xy 181.61 78.74) (xy 205.74 78.74))
     (stroke (width 0) (type default))
@@
   )
   (wire (pts (xy 158.75 162.56) (xy 163.83 162.56))
+    (stroke (width 0) (type default))
+  )
+  (wire (pts (xy 252.73 45.72) (xy 252.73 53.34))
     (stroke (width 0) (type default))
   )
@@
   )
   (text "VOUT\n" (at 274.32 44.45 0)
-    (effects (font (size 1.27 1.27)) (justify left bottom))
-  )
-  (label "AVIN (LMS)" (at 100.33 69.85 0) (fields_autoplaced)
     (effects (font (size 1.27 1.27)) (justify left bottom))
   )
@@
     )
   )
+  (global_label "3V3_REF" (shape input) (at 252.73 45.72 0) (fields_autoplaced)
+    (effects (font (size 1.27 1.27)) (justify left))
+    (property "Intersheetrefs" "${INTERSHEET_REFS}" (at 263.698 45.72 0)
+      (effects (font (size 1.27 1.27)) (justify left) hide)
+    )
+  )
   (global_label "AWR_GPIO_3" (shape input) (at 34.29 124.46 180) (fields_autoplaced)
     (effects (font (size 1.27 1.27)) (justify right))
@@
     )
   )
-  (global_label "1V2" (shape input) (at 71.12 149.86 180) (fields_autoplaced)
+  (global_label "1V24" (shape input) (at 71.12 149.86 180) (fields_autoplaced)
     (effects (font (size 1.27 1.27)) (justify right))
-    (property "Intersheetrefs" "${INTERSHEET_REFS}" (at 64.6272 149.86 0)
+    (property "Intersheetrefs" "${INTERSHEET_REFS}" (at 63.4177 149.86 0)
       (effects (font (size 1.27 1.27)) (justify right) hide)
     )
@@
   (symbol (lib_id "Device:C_Small") (at 83.82 146.05 0) (unit 1)
     (in_bom yes) (on_board yes) (dnp no)
-    (property "Reference" "C38" (at 78.74 146.05 0)
+    (property "Reference" "C38" (at 77.47 146.05 0)
       (effects (font (size 1.27 1.27)) (justify left))
     )
@@
         )
       )
+    )
+  )
+  (symbol (lib_id "power:+5V") (at 100.33 69.85 0) (unit 1)
+    (in_bom yes) (on_board yes) (dnp no) (fields_autoplaced)
+    (property "Reference" "#PWR056" (at 100.33 73.66 0)
+      (effects (font (size 1.27 1.27)) hide)
+    )
+    (property "Value" "+5V" (at 100.33 64.77 0)
+      (effects (font (size 1.27 1.27)))
+    )
+    (property "Footprint" "" (at 100.33 69.85 0)
+      (effects (font (size 1.27 1.27)) hide)
+    )
+    (property "Datasheet" "" (at 100.33 69.85 0)
+      (effects (font (size 1.27 1.27)) hide)
+    )
+    (pin "1")
+    (instances
+      (project "radar"
+        (path "/88b309aa-5f0e-45d7-beec-81d4b0ee2121/7a3c78f1-80f2-463b-a37f-9a7b3cc7f964/62900e5d-413e-4591-98ac-b12b6d69be62"
+          (reference "#PWR056") (unit 1)
+        )
+      )
