File: stepdwn_and_ldo.kicad_sch (KiCad schematic)
At the start: 48 parts, among them J1 USB_C_Receptacle_USB2.0_14P, U2 BQ25895RTW, U4 PTPS7A5310AQWRTJQ1, U5 LMS36353QRNLRQ1

Commit message: finding exact crystal used in ref design, finishing shcematics
Connections:
- net AWR_RESET renamed AWR_NRESET
Changed lines of the file:
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@@
+    (effects (font (size 1.27 1.27)) (justify left bottom))
+  )
+  (label "PMID" (at 245.11 20.32 0) (fields_autoplaced)
     (effects (font (size 1.27 1.27)) (justify left bottom))
   )
@@
     (property "Intersheetrefs" "${INTERSHEET_REFS}" (at 93.98 135.1257 90)
       (effects (font (size 1.27 1.27)) (justify right) hide)
-    )
-  )
-  (global_label "PMID" (shape input) (at 245.11 20.32 0) (fields_autoplaced)
-    (effects (font (size 1.27 1.27)) (justify left))
-    (property "Intersheetrefs" "${INTERSHEET_REFS}" (at 252.6914 20.32 0)
-      (effects (font (size 1.27 1.27)) (justify left) hide)
     )
   )
@@
     )
   )
-  (global_label "AWR_RESET" (shape input) (at 218.44 80.01 0) (fields_autoplaced)
+  (global_label "AWR_NRESET" (shape input) (at 218.44 80.01 0) (fields_autoplaced)
     (effects (font (size 1.27 1.27)) (justify left))
-    (property "Intersheetrefs" "${INTERSHEET_REFS}" (at 231.9479 80.01 0)
+    (property "Intersheetrefs" "${INTERSHEET_REFS}" (at 233.2784 80.01 0)
       (effects (font (size 1.27 1.27)) (justify left) hide)
     )

Commit message: squashing ERC errors
Other:
- note removed: "This may be renamed once reset pin on AWR is declared"
Changed lines of the file:
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@@
-    (effects (font (size 1.27 1.27)) (justify left bottom))
-  )
-  (text "This may be renamed once\nreset pin on AWR is declared\n"
-    (at 213.36 86.36 0)
     (effects (font (size 1.27 1.27)) (justify left bottom))
   )

Commit message: squashed ERC errors, moving onto pcb, grabbing fuse footprint
Parts:
- removed R28: 10k, symbol Device:R_Small_US
- added R36: 10k, symbol Device:R_Small_US
Connections:
- net PMID is gone; now on net +5V: F1.2
- net SYS: now also C42.2, L4.2, U2.15 (SYS), U2.16 (SYS), R36.2
- net at U2.8 (OTG): now also R36.1
Changed lines of the file:
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@@
   (junction (at 133.35 55.88) (diameter 0) (color 0 0 0 0)
+  )
+  (junction (at 97.79 73.66) (diameter 0) (color 0 0 0 0)
   )
   (junction (at 172.72 162.56) (diameter 0) (color 0 0 0 0)
@@
     (stroke (width 0) (type default))
   )
-  (wire (pts (xy 49.53 106.68) (xy 58.42 106.68))
+  (wire (pts (xy 53.34 106.68) (xy 58.42 106.68))
     (stroke (width 0) (type default))
   )
@@
     (stroke (width 0) (type default))
   )
-  (wire (pts (xy 45.72 119.38) (xy 45.72 127))
-    (stroke (width 0) (type default))
-  )
   (wire (pts (xy 205.74 91.44) (xy 205.74 93.98))
     (stroke (width 0) (type default))
@@
     (stroke (width 0) (type default))
   )
+  (wire (pts (xy 97.79 73.66) (xy 107.95 73.66))
+    (stroke (width 0) (type default))
+  )
   (wire (pts (xy 45.72 161.29) (xy 59.69 161.29))
     (stroke (width 0) (type default))
@@
     (stroke (width 0) (type default))
   )
-  (wire (pts (xy 49.53 109.22) (xy 45.72 109.22))
+  (wire (pts (xy 49.53 110.49) (xy 53.34 110.49))
     (stroke (width 0) (type default))
   )
@@
     (stroke (width 0) (type default))
   )
+  (wire (pts (xy 102.87 66.04) (xy 102.87 62.23))
+    (stroke (width 0) (type default))
+  )
   (wire (pts (xy 194.31 31.75) (xy 209.55 31.75))
     (stroke (width 0) (type default))
@@
     (stroke (width 0) (type default))
   )
-  (wire (pts (xy 90.17 72.39) (xy 100.33 72.39))
+  (wire (pts (xy 90.17 73.66) (xy 97.79 73.66))
     (stroke (width 0) (type default))
   )
@@
     (stroke (width 0) (type default))
   )
-  (wire (pts (xy 90.17 76.2) (xy 90.17 72.39))
+  (wire (pts (xy 90.17 76.2) (xy 90.17 73.66))
     (stroke (width 0) (type default))
   )
@@
     (stroke (width 0) (type default))
   )
+  (wire (pts (xy 97.79 73.66) (xy 97.79 66.04))
+    (stroke (width 0) (type default))
+  )
   (wire (pts (xy 93.98 185.42) (xy 95.25 185.42))
     (stroke (width 0) (type default))
@@
     (stroke (width 0) (type default))
   )
+  (wire (pts (xy 38.1 110.49) (xy 44.45 110.49))
+    (stroke (width 0) (type default))
+  )
   (wire (pts (xy 194.31 26.67) (xy 194.31 31.75))
     (stroke (width 0) (type default))
   )
-  (wire (pts (xy 100.33 72.39) (xy 100.33 69.85))
+  (wire (pts (xy 107.95 73.66) (xy 107.95 71.12))
     (stroke (width 0) (type default))
   )
@@
     (stroke (width 0) (type default))
   )
+  (wire (pts (xy 97.79 66.04) (xy 102.87 66.04))
+    (stroke (width 0) (type default))
+  )
   (wire (pts (xy 160.02 114.3) (xy 205.74 114.3))
     (stroke (width 0) (type default))
@@
     (stroke (width 0) (type default))
   )
-  (wire (pts (xy 45.72 109.22) (xy 45.72 114.3))
-    (stroke (width 0) (type default))
-  )
   (wire (pts (xy 133.35 48.26) (xy 133.35 45.72))
     (stroke (width 0) (type default))
@@
     (stroke (width 0) (type default))
   )
-  (wire (pts (xy 49.53 109.22) (xy 49.53 106.68))
+  (wire (pts (xy 53.34 110.49) (xy 53.34 106.68))
     (stroke (width 0) (type default))
   )
@@
     (effects (font (size 1.27 1.27)) (justify left bottom))
   )
-  (label "PMID" (at 245.11 20.32 0) (fields_autoplaced)
+  (label "PMID" (at 238.76 20.32 0) (fields_autoplaced)
     (effects (font (size 1.27 1.27)) (justify left bottom))
   )
-  (label "SYS" (at 45.72 127 0) (fields_autoplaced)
+  (label "SYS" (at 83.82 91.44 0) (fields_autoplaced)
+    (effects (font (size 1.27 1.27)) (justify left bottom))
+  )
+  (label "PMID" (at 100.33 73.66 0) (fields_autoplaced)
+    (effects (font (size 1.27 1.27)) (justify left bottom))
+  )
+  (label "SYS" (at 38.1 110.49 0) (fields_autoplaced)
     (effects (font (size 1.27 1.27)) (justify left bottom))
   )
@@
     (effects (font (size 1.27 1.27)) (justify right))
     (property "Intersheetrefs" "${INTERSHEET_REFS}" (at 30.5791 97.79 0)
+      (effects (font (size 1.27 1.27)) (justify right) hide)
+    )
+  )
+  (global_label "PMID" (shape bidirectional) (at 102.87 62.23 180) (fields_autoplaced)
+    (effects (font (size 1.27 1.27)) (justify right))
+    (property "Intersheetrefs" "${INTERSHEET_REFS}" (at 94.1773 62.23 0)
       (effects (font (size 1.27 1.27)) (justify right) hide)
     )
@@
         (path "/88b309aa-5f0e-45d7-beec-81d4b0ee2121/7a3c78f1-80f2-463b-a37f-9a7b3cc7f964/62900e5d-413e-4591-98ac-b12b6d69be62"
           (reference "#PWR011") (unit 1)
-        )
-      )
-    )
-  )
-  (symbol (lib_id "Device:R_Small_US") (at 45.72 116.84 180) (unit 1)
-    (in_bom yes) (on_board yes) (dnp no) (fields_autoplaced)
-    (property "Reference" "R28" (at 48.26 115.57 0)
-      (effects (font (size 1.27 1.27)) (justify right))
-    )
-    (property "Value" "10k" (at 48.26 118.11 0)
-      (effects (font (size 1.27 1.27)) (justify right))
-    )
-    (property "Footprint" "" (at 45.72 116.84 0)
-      (effects (font (size 1.27 1.27)) hide)
-    )
-    (property "Datasheet" "~" (at 45.72 116.84 0)
-      (effects (font (size 1.27 1.27)) hide)
-    )
-    (pin "2")
-    (pin "1")
-    (instances
-      (project "radar"
-        (path "/88b309aa-5f0e-45d7-beec-81d4b0ee2121/7a3c78f1-80f2-463b-a37f-9a7b3cc7f964/62900e5d-413e-4591-98ac-b12b6d69be62"
-          (reference "R28") (unit 1)
         )
       )
@@
     )
   )
-  (symbol (lib_id "power:+5V") (at 100.33 69.85 0) (unit 1)
-    (in_bom yes) (on_board yes) (dnp no) (fields_autoplaced)
-    (property "Reference" "#PWR056" (at 100.33 73.66 0)
-      (effects (font (size 1.27 1.27)) hide)
-    )
-    (property "Value" "+5V" (at 100.33 64.77 0)
-      (effects (font (size 1.27 1.27)))
-    )
-    (property "Footprint" "" (at 100.33 69.85 0)
-      (effects (font (size 1.27 1.27)) hide)
-    )
-    (property "Datasheet" "" (at 100.33 69.85 0)
+  (symbol (lib_id "power:+5V") (at 107.95 71.12 0) (unit 1)
+    (in_bom yes) (on_board yes) (dnp no) (fields_autoplaced)
+    (property "Reference" "#PWR056" (at 107.95 74.93 0)
+      (effects (font (size 1.27 1.27)) hide)
+    )
+    (property "Value" "+5V" (at 107.95 66.04 0)
+      (effects (font (size 1.27 1.27)))
+    )
+    (property "Footprint" "" (at 107.95 71.12 0)
+      (effects (font (size 1.27 1.27)) hide)
+    )
+    (property "Datasheet" "" (at 107.95 71.12 0)
       (effects (font (size 1.27 1.27)) hide)
     )
@@
         (path "/88b309aa-5f0e-45d7-beec-81d4b0ee2121/7a3c78f1-80f2-463b-a37f-9a7b3cc7f964/62900e5d-413e-4591-98ac-b12b6d69be62"
           (reference "R11") (unit 1)
+        )
+      )
+    )
+  )
+  (symbol (lib_id "power:+5V") (at 245.11 20.32 0) (unit 1)
+    (in_bom yes) (on_board yes) (dnp no) (fields_autoplaced)
+    (property "Reference" "#PWR019" (at 245.11 24.13 0)
+      (effects (font (size 1.27 1.27)) hide)
+    )
+    (property "Value" "+5V" (at 245.11 15.24 0)
+      (effects (font (size 1.27 1.27)))
+    )
+    (property "Footprint" "" (at 245.11 20.32 0)
+      (effects (font (size 1.27 1.27)) hide)
+    )
+    (property "Datasheet" "" (at 245.11 20.32 0)
+      (effects (font (size 1.27 1.27)) hide)
+    )
+    (pin "1")
+    (instances
+      (project "radar"
+        (path "/88b309aa-5f0e-45d7-beec-81d4b0ee2121/7a3c78f1-80f2-463b-a37f-9a7b3cc7f964/62900e5d-413e-4591-98ac-b12b6d69be62"
+          (reference "#PWR019") (unit 1)
         )
       )
@@
         )
       )
+    )
+  )
+  (symbol (lib_id "Device:R_Small_US") (at 46.99 110.49 270) (unit 1)
+    (in_bom yes) (on_board yes) (dnp no)
+    (property "Reference" "R36" (at 44.45 111.76 90)
+      (effects (font (size 1.27 1.27)))
+    )
+    (property "Value" "10k" (at 50.8 111.76 90)
+      (effects (font (size 1.27 1.27)))
+    )
+    (property "Footprint" "" (at 46.99 110.49 0)
+      (effects (font (size 1.27 1.27)) hide)
+    )
+    (property "Datasheet" "~" (at 46.99 110.49 0)
+      (effects (font (size 1.27 1.27)) hide)
+    )
+    (pin "2")
+    (pin "1")
+    (instances
+      (project "radar"
+        (path "/88b309aa-5f0e-45d7-beec-81d4b0ee2121/7a3c78f1-80f2-463b-a37f-9a7b3cc7f964/62900e5d-413e-4591-98ac-b12b6d69be62"
+          (reference "R36") (unit 1)
+        )
+      )

Commit message: adding footprints
Parts:
- removed C35: 0.1muF, symbol Device:C_Small
- removed C36: 22muF, symbol Device:C_Small
- removed F1: 5A, symbol Device:Fuse
- removed J1: USB_C_Receptacle_USB2.0_14P, symbol Connector:USB_C_Receptacle_USB2.0_14P
- removed R10, R11: 5k, symbol Device:R_Small_US
- added F2: Polyfuse, MF_LSMF330:MFLSM, symbol Device:Polyfuse
- BT1: footprint (none) -> MF_LSMF330:MFLSM
- C32, C33, C34, C37, C38, C39, C40, C42, C43, C45, C46, C47, C48, C49, C5, C50, C51, C52, C53, C54, C55, C56, C57, C58, C7: footprint (none) -> Capacitor_SMD:C_0603_1608Metric
- C6: footprint (none) -> Capacitor_SMD:C_0402_1005Metric
- L4, L5, L6: footprint (none) -> Inductor_SMD:L_0603_1608Metric
- R16, R17, R18, R19, R20, R21, R23, R36: footprint (none) -> Resistor_SMD:R_0603_1608Metric
Connections:
- net +5V: now also F2.1
- net at C51.1, C53.1, C55.1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: now also F2.2
- net VBUS: now reaches U2.1 (VBUS)
- net D+: now reaches U2.2 (D+)
- net D-: now reaches U2.3 (D-)
- no-connect marks 5 -> 3
Other:
- moved on the sheet: BT1, C39, C40, C42, C5, C6, L4, R16, R17, R18, R19, R20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
