File: decoup_caps.kicad_sch (KiCad schematic)
At the start: 26 parts

Commit message: adding footprints
Parts:
- C13, C14, C15, C16, C17, C18, C19, C20, C41, C44, C59, C60, C61, C62, C63, C64, C65, C66, C67, C68, C69, C70, C71, C72, C73, C74: footprint (none) -> Capacitor_SMD:C_0603_1608Metric
Changed lines of the file:
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@@
       (effects (font (size 1.27 1.27)) (justify left))
     )
-    (property "Footprint" "" (at 260.0452 48.26 0)
+    (property "Footprint" "Capacitor_SMD:C_0603_1608Metric" (at 260.0452 48.26 0)
       (effects (font (size 1.27 1.27)) hide)
     )
@@
       (effects (font (size 1.27 1.27)) (justify left))
     )
-    (property "Footprint" "" (at 152.0952 101.6 0)
+    (property "Footprint" "Capacitor_SMD:C_0603_1608Metric" (at 152.0952 101.6 0)
       (effects (font (size 1.27 1.27)) hide)
     )
@@
       (effects (font (size 1.27 1.27)) (justify left))
     )
-    (property "Footprint" "" (at 219.4052 48.26 0)
+    (property "Footprint" "Capacitor_SMD:C_0603_1608Metric" (at 219.4052 48.26 0)
       (effects (font (size 1.27 1.27)) hide)
     )
@@
       (effects (font (size 1.27 1.27)) (justify left))
     )
-    (property "Footprint" "" (at 21.2852 49.53 0)
+    (property "Footprint" "Capacitor_SMD:C_0603_1608Metric" (at 21.2852 49.53 0)
       (effects (font (size 1.27 1.27)) hide)
     )
@@
       (effects (font (size 1.27 1.27)) (justify left))
     )
-    (property "Footprint" "" (at 199.0852 92.71 0)
+    (property "Footprint" "Capacitor_SMD:C_0603_1608Metric" (at 199.0852 92.71 0)
       (effects (font (size 1.27 1.27)) hide)
     )
@@
       (effects (font (size 1.27 1.27)) (justify left))
     )
-    (property "Footprint" "" (at 101.2952 104.14 0)
+    (property "Footprint" "Capacitor_SMD:C_0603_1608Metric" (at 101.2952 104.14 0)
       (effects (font (size 1.27 1.27)) hide)
     )
@@
       (effects (font (size 1.27 1.27)) (justify left))
     )
-    (property "Footprint" "" (at 148.2852 148.59 0)
+    (property "Footprint" "Capacitor_SMD:C_0603_1608Metric" (at 148.2852 148.59 0)
       (effects (font (size 1.27 1.27)) hide)
     )
@@
       (effects (font (size 1.27 1.27)) (justify left))
     )
-    (property "Footprint" "" (at 171.1452 101.6 0)
+    (property "Footprint" "Capacitor_SMD:C_0603_1608Metric" (at 171.1452 101.6 0)
       (effects (font (size 1.27 1.27)) hide)
     )
@@
       (effects (font (size 1.27 1.27)) (justify left))
     )
-    (property "Footprint" "" (at 80.9752 162.56 0)
+    (property "Footprint" "Capacitor_SMD:C_0603_1608Metric" (at 80.9752 162.56 0)
       (effects (font (size 1.27 1.27)) hide)
     )
@@
       (effects (font (size 1.27 1.27)) (justify left))
     )
-    (property "Footprint" "" (at 188.9252 46.99 0)
+    (property "Footprint" "Capacitor_SMD:C_0603_1608Metric" (at 188.9252 46.99 0)
       (effects (font (size 1.27 1.27)) hide)
     )
@@
       (effects (font (size 1.27 1.27)) (justify left))
     )
-    (property "Footprint" "" (at 187.6552 148.59 0)
+    (property "Footprint" "Capacitor_SMD:C_0603_1608Metric" (at 187.6552 148.59 0)
       (effects (font (size 1.27 1.27)) hide)
     )
@@
       (effects (font (size 1.27 1.27)) (justify left))
     )
-    (property "Footprint" "" (at 167.3352 148.59 0)
+    (property "Footprint" "Capacitor_SMD:C_0603_1608Metric" (at 167.3352 148.59 0)
       (effects (font (size 1.27 1.27)) hide)
     )
@@
       (effects (font (size 1.27 1.27)) (justify left))
     )
-    (property "Footprint" "" (at 105.1052 48.26 0)
+    (property "Footprint" "Capacitor_SMD:C_0603_1608Metric" (at 105.1052 48.26 0)
       (effects (font (size 1.27 1.27)) hide)
     )
@@
       (effects (font (size 1.27 1.27)) (justify left))
     )
-    (property "Footprint" "" (at 135.5852 101.6 0)
+    (property "Footprint" "Capacitor_SMD:C_0603_1608Metric" (at 135.5852 101.6 0)
       (effects (font (size 1.27 1.27)) hide)
     )
@@
       (effects (font (size 1.27 1.27)) (justify left))
     )
-    (property "Footprint" "" (at 33.9852 49.53 0)
+    (property "Footprint" "Capacitor_SMD:C_0603_1608Metric" (at 33.9852 49.53 0)
       (effects (font (size 1.27 1.27)) hide)
     )
@@
       (effects (font (size 1.27 1.27)) (justify left))
     )
-    (property "Footprint" "" (at 53.0352 104.14 0)
+    (property "Footprint" "Capacitor_SMD:C_0603_1608Metric" (at 53.0352 104.14 0)
       (effects (font (size 1.27 1.27)) hide)
     )
@@
       (effects (font (size 1.27 1.27)) (justify left))
     )
-    (property "Footprint" "" (at 50.4952 49.53 0)
+    (property "Footprint" "Capacitor_SMD:C_0603_1608Metric" (at 50.4952 49.53 0)
       (effects (font (size 1.27 1.27)) hide)
     )
@@
       (effects (font (size 1.27 1.27)) (justify left))
     )
-    (property "Footprint" "" (at 36.5252 161.29 0)
+    (property "Footprint" "Capacitor_SMD:C_0603_1608Metric" (at 36.5252 161.29 0)
       (effects (font (size 1.27 1.27)) hide)
     )
@@
       (effects (font (size 1.27 1.27)) (justify left))
     )
-    (property "Footprint" "" (at 243.5352 48.26 0)
+    (property "Footprint" "Capacitor_SMD:C_0603_1608Metric" (at 243.5352 48.26 0)
       (effects (font (size 1.27 1.27)) hide)
     )
@@
       (effects (font (size 1.27 1.27)) (justify left))
     )
-    (property "Footprint" "" (at 131.7752 148.59 0)
+    (property "Footprint" "Capacitor_SMD:C_0603_1608Metric" (at 131.7752 148.59 0)
       (effects (font (size 1.27 1.27)) hide)
     )
@@
       (effects (font (size 1.27 1.27)) (justify left))
     )
-    (property "Footprint" "" (at 235.9152 93.98 0)
+    (property "Footprint" "Capacitor_SMD:C_0603_1608Metric" (at 235.9152 93.98 0)
       (effects (font (size 1.27 1.27)) hide)
     )
@@
       (effects (font (size 1.27 1.27)) (justify left))
     )
-    (property "Footprint" "" (at 84.7852 104.14 0)
+    (property "Footprint" "Capacitor_SMD:C_0603_1608Metric" (at 84.7852 104.14 0)
       (effects (font (size 1.27 1.27)) hide)
     )
@@
       (effects (font (size 1.27 1.27)) (justify left))
     )
-    (property "Footprint" "" (at 172.4152 46.99 0)
+    (property "Footprint" "Capacitor_SMD:C_0603_1608Metric" (at 172.4152 46.99 0)
       (effects (font (size 1.27 1.27)) hide)
     )
@@
       (effects (font (size 1.27 1.27)) (justify left))
     )
-    (property "Footprint" "" (at 139.3952 52.07 0)
+    (property "Footprint" "Capacitor_SMD:C_0603_1608Metric" (at 139.3952 52.07 0)
       (effects (font (size 1.27 1.27)) hide)
     )
@@
       (effects (font (size 1.27 1.27)) (justify left))
     )
-    (property "Footprint" "" (at 36.5252 104.14 0)
+    (property "Footprint" "Capacitor_SMD:C_0603_1608Metric" (at 36.5252 104.14 0)
       (effects (font (size 1.27 1.27)) hide)
     )
@@
       (effects (font (size 1.27 1.27)) (justify left))
     )
-    (property "Footprint" "" (at 73.3552 49.53 0)
-      (effects (font (size 1.27 1.27)) hide)
-    )
+    (property "Footprint" "Capacitor_SMD:C_0603_1608Metric" (at 73.3552 49.53 0)
+      (effects (font (size 1.27 1.27)) hide)
+    )
