File: pmics.kicad_sch (KiCad schematic)
At the start: 89 parts, among them IC1 BQ25713RSNR, IC2 TPS54540DDA, IC3 TPS54540DDA, Q1 CSD17308Q3, Q2 CSD17308Q3, Q3 CSD17308Q3, Q4 CSD17308Q3, Q5 CSD25404Q3

Commit message: finishing mcu design schematic
Connections:
- net GND: now also IC1.14 (CMPIN)
- net CHRG_OK renamed BQ_CHRG_OK
- net ST_SCL renamed BQ_SCL
- net ST_SDA renamed BQ_SDA
- no-connect marks 2 -> 1
Changed lines of the file:
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@@
   (junction (at 350.52 46.99) (diameter 0) (color 0 0 0 0)
   )
-  (no_connect (at 125.73 107.95))
   (no_connect (at 125.73 104.14))
   (wire (pts (xy 87.63 226.06) (xy 92.71 226.06))
@@
     (stroke (width 0) (type default))
   )
+  (wire (pts (xy 138.43 114.3) (xy 140.97 114.3))
+    (stroke (width 0) (type default))
+  )
   (wire (pts (xy 60.96 83.82) (xy 60.96 86.36))
     (stroke (width 0) (type default))
@@
     (stroke (width 0) (type default))
   )
+  (wire (pts (xy 125.73 107.95) (xy 138.43 107.95))
+    (stroke (width 0) (type default))
+  )
   (wire (pts (xy 167.64 113.03) (xy 179.07 113.03))
     (stroke (width 0) (type default))
@@
   )
   (wire (pts (xy 335.28 218.44) (xy 335.28 213.36))
+    (stroke (width 0) (type default))
+  )
+  (wire (pts (xy 138.43 107.95) (xy 138.43 114.3))
     (stroke (width 0) (type default))
   )
@@
     )
   )
-  (global_label "ST_SDA" (shape bidirectional) (at 127 115.57 0) (fields_autoplaced)
+  (global_label "BQ_SDA" (shape bidirectional) (at 127 115.57 0) (fields_autoplaced)
     (effects (font (size 1.27 1.27)) (justify left))
-    (property "Intersheetrefs" "${INTERSHEET_REFS}" (at 137.8093 115.57 0)
+    (property "Intersheetrefs" "${INTERSHEET_REFS}" (at 138.2327 115.57 0)
       (effects (font (size 1.27 1.27)) (justify left) hide)
     )
   )
-  (global_label "ST_SCL" (shape bidirectional) (at 127 111.76 0) (fields_autoplaced)
+  (global_label "BQ_SCL" (shape bidirectional) (at 127 111.76 0) (fields_autoplaced)
     (effects (font (size 1.27 1.27)) (justify left))
-    (property "Intersheetrefs" "${INTERSHEET_REFS}" (at 137.7488 111.76 0)
+    (property "Intersheetrefs" "${INTERSHEET_REFS}" (at 138.1722 111.76 0)
       (effects (font (size 1.27 1.27)) (justify left) hide)
     )
@@
     )
   )
-  (global_label "CHRG_OK" (shape bidirectional) (at 77.47 111.76 180) (fields_autoplaced)
+  (global_label "BQ_CHRG_OK" (shape bidirectional) (at 77.47 111.76 180) (fields_autoplaced)
     (effects (font (size 1.27 1.27)) (justify right))
-    (property "Intersheetrefs" "${INTERSHEET_REFS}" (at 64.6649 111.76 0)
+    (property "Intersheetrefs" "${INTERSHEET_REFS}" (at 61.0968 111.76 0)
       (effects (font (size 1.27 1.27)) (justify right) hide)
     )

Commit message: adding prochot to design, clearing ERC
Parts:
- added R37: 10m, Resistor_SMD:R_0603_1608Metric, symbol Device:R_Small_US
Connections:
- net GND: now also R37.1; no longer C21.2, Q1.5 (D_1), Q1.6 (D_2), Q1.7 (D_3), Q1.8 (D_4), Q1.9 (D_5), R14.2
- net at C30.2, C31.2, Q5.1 (D_1)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: now also Q5.2 (D_2), Q5.3 (D_3)
- net BQ_PROCHOT: now reaches IC1.11 (~{PROCHOT})
- new net: C21.2, Q1.5 (D_1), Q1.6 (D_2), Q1.7 (D_3), Q1.8 (D_4), Q1.9 (D_5), R14.2, R37.2
Changed lines of the file:
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@@
   (junction (at 292.1 107.95) (diameter 0) (color 0 0 0 0)
   )
+  (junction (at 302.26 217.17) (diameter 0) (color 0 0 0 0)
+  )
   (junction (at 261.62 219.71) (diameter 0) (color 0 0 0 0)
   )
@@
   )
   (junction (at 203.2 213.36) (diameter 0) (color 0 0 0 0)
+  )
+  (junction (at 302.26 219.71) (diameter 0) (color 0 0 0 0)
   )
   (junction (at 326.39 127) (diameter 0) (color 0 0 0 0)
@@
     (stroke (width 0) (type default))
   )
+  (wire (pts (xy 130.81 119.38) (xy 130.81 125.73))
+    (stroke (width 0) (type default))
+  )
   (wire (pts (xy 66.04 222.25) (xy 67.31 222.25))
     (stroke (width 0) (type default))
@@
     (stroke (width 0) (type default))
   )
-  (wire (pts (xy 86.36 213.36) (xy 96.52 213.36))
+  (wire (pts (xy 86.36 213.36) (xy 88.9 213.36))
     (stroke (width 0) (type default))
   )
@@
     (stroke (width 0) (type default))
   )
+  (wire (pts (xy 302.26 219.71) (xy 302.26 222.25))
+    (stroke (width 0) (type default))
+  )
   (wire (pts (xy 226.06 49.53) (xy 234.95 49.53))
     (stroke (width 0) (type default))
@@
     (stroke (width 0) (type default))
   )
+  (wire (pts (xy 302.26 217.17) (xy 302.26 219.71))
+    (stroke (width 0) (type default))
+  )
   (wire (pts (xy 59.69 240.03) (xy 59.69 231.14))
     (stroke (width 0) (type default))
@@
     (stroke (width 0) (type default))
   )
+  (wire (pts (xy 93.98 213.36) (xy 96.52 213.36))
+    (stroke (width 0) (type default))
+  )
   (wire (pts (xy 115.57 213.36) (xy 125.73 213.36))
     (stroke (width 0) (type default))
@@
     (stroke (width 0) (type default))
   )
+  (wire (pts (xy 125.73 119.38) (xy 130.81 119.38))
+    (stroke (width 0) (type default))
+  )
   (wire (pts (xy 295.91 193.04) (xy 295.91 191.77))
     (stroke (width 0) (type default))
@@
   )
   (wire (pts (xy 259.08 140.97) (xy 250.19 140.97))
+    (stroke (width 0) (type default))
+  )
+  (wire (pts (xy 130.81 125.73) (xy 151.13 125.73))
     (stroke (width 0) (type default))
   )
@@
     (property "Intersheetrefs" "${INTERSHEET_REFS}" (at 30.7378 213.36 0)
       (effects (font (size 1.27 1.27)) (justify right) hide)
+    )
+  )
+  (global_label "BQ_PROCHOT" (shape bidirectional) (at 151.13 125.73 0) (fields_autoplaced)
+    (effects (font (size 1.27 1.27)) (justify left))
+    (property "Intersheetrefs" "${INTERSHEET_REFS}" (at 167.5637 125.73 0)
+      (effects (font (size 1.27 1.27)) (justify left) hide)
     )
   )
@@
         )
       )
+    )
+  )
+  (symbol (lib_id "Device:R_Small_US") (at 91.44 213.36 90) (unit 1)
+    (in_bom yes) (on_board yes) (dnp no)
+    (property "Reference" "R37" (at 90.17 208.28 90)
+      (effects (font (size 1.27 1.27)) (justify right))
+    )
+    (property "Value" "10m" (at 90.17 210.82 90)
+      (effects (font (size 1.27 1.27)) (justify right))
+    )
+    (property "Footprint" "Resistor_SMD:R_0603_1608Metric" (at 91.44 213.36 0)
+      (effects (font (size 1.27 1.27)) hide)
+    )
+    (property "Datasheet" "~" (at 91.44 213.36 0)
+      (effects (font (size 1.27 1.27)) hide)
+    )
+    (pin "1")
+    (pin "2")
+    (instances
+      (project "radar2"
+        (path "/4b235fed-a05d-46ae-99fd-4a907d865754/3b0f6a2d-e812-480b-87fe-92eb8a340c39"
+          (reference "R37") (unit 1)
+        )
+      )

Commit message: adding all footprints moving onto pcb
Parts:
- C13, C14, C15, C16, C17, C24, C25, C26, C27, C28: value 10uF -> 0.1uF
- L1, L2, L3: footprint (none) -> Inductor_SMD:L_0603_1608Metric
- R19, R20, R21, R22, R23, R24, R25, R26, R27, R28, R29, R30: footprint (none) -> Resistor_SMD:R_0603_1608Metric
Changed lines of the file:
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@@
   (junction (at 308.61 52.07) (diameter 0) (color 0 0 0 0)
   )
+  (junction (at 59.69 265.43) (diameter 0) (color 0 0 0 0)
+  )
   (junction (at 344.17 124.46) (diameter 0) (color 0 0 0 0)
   )
@@
   (junction (at 276.86 219.71) (diameter 0) (color 0 0 0 0)
   )
-  (junction (at 59.69 266.7) (diameter 0) (color 0 0 0 0)
-  )
   (junction (at 162.56 224.79) (diameter 0) (color 0 0 0 0)
   )
@@
     (stroke (width 0) (type default))
   )
-  (wire (pts (xy 59.69 257.81) (xy 59.69 266.7))
+  (wire (pts (xy 59.69 257.81) (xy 59.69 265.43))
     (stroke (width 0) (type default))
   )
@@
     (stroke (width 0) (type default))
   )
-  (wire (pts (xy 59.69 266.7) (xy 53.34 266.7))
+  (wire (pts (xy 59.69 265.43) (xy 53.34 265.43))
     (stroke (width 0) (type default))
   )
@@
     (stroke (width 0) (type default))
   )
+  (wire (pts (xy 59.69 265.43) (xy 59.69 266.7))
+    (stroke (width 0) (type default))
+  )
   (wire (pts (xy 93.98 213.36) (xy 96.52 213.36))
     (stroke (width 0) (type default))
@@
       (effects (font (size 1.27 1.27)) (justify left))
     )
-    (property "Value" "10uF" (at 302.26 196.85 0)
+    (property "Value" "0.1uF" (at 302.26 196.85 0)
       (effects (font (size 1.27 1.27)) (justify left))
     )
@@
       (effects (font (size 1.27 1.27)) (justify left))
     )
-    (property "Value" "10uF" (at 60.96 228.6 90)
+    (property "Value" "0.1uF" (at 60.96 228.6 90)
       (effects (font (size 1.27 1.27)) (justify left))
     )
@@
       (effects (font (size 1.27 1.27)))
     )
-    (property "Footprint" "" (at 194.31 213.36 0)
+    (property "Footprint" "Inductor_SMD:L_0603_1608Metric" (at 194.31 213.36 0)
       (effects (font (size 1.27 1.27)) hide)
     )
@@
       (effects (font (size 1.27 1.27)) (justify left))
     )
-    (property "Value" "10uF" (at 60.96 237.49 90)
+    (property "Value" "0.1uF" (at 60.96 237.49 90)
       (effects (font (size 1.27 1.27)) (justify left))
     )
@@
       (effects (font (size 1.27 1.27)) (justify left))
     )
-    (property "Footprint" "" (at 350.52 54.61 0)
+    (property "Footprint" "Resistor_SMD:R_0603_1608Metric" (at 350.52 54.61 0)
       (effects (font (size 1.27 1.27)) hide)
     )
@@
       (effects (font (size 1.27 1.27)) (justify left))
     )
-    (property "Footprint" "" (at 250.19 147.32 0)
+    (property "Footprint" "Resistor_SMD:R_0603_1608Metric" (at 250.19 147.32 0)
       (effects (font (size 1.27 1.27)) hide)
     )
@@
       (effects (font (size 1.27 1.27)))
     )
-    (property "Footprint" "" (at 304.8 107.95 0)
+    (property "Footprint" "Inductor_SMD:L_0603_1608Metric" (at 304.8 107.95 0)
       (effects (font (size 1.27 1.27)) hide)
     )
@@
       (effects (font (size 1.27 1.27)))
     )
-    (property "Footprint" "" (at 311.15 30.48 0)
+    (property "Footprint" "Inductor_SMD:L_0603_1608Metric" (at 311.15 30.48 0)
       (effects (font (size 1.27 1.27)) hide)
     )
@@
       (effects (font (size 1.27 1.27)) (justify left))
     )
-    (property "Footprint" "" (at 302.26 138.43 0)
+    (property "Footprint" "Resistor_SMD:R_0603_1608Metric" (at 302.26 138.43 0)
       (effects (font (size 1.27 1.27)) hide)
     )
@@
       (effects (font (size 1.27 1.27)) (justify left))
     )
-    (property "Value" "10uF" (at 62.23 246.38 90)
+    (property "Value" "0.1uF" (at 62.23 246.38 90)
       (effects (font (size 1.27 1.27)) (justify left))
     )
@@
       (effects (font (size 1.27 1.27)) (justify left))
     )
-    (property "Value" "10uF" (at 60.96 255.27 90)
+    (property "Value" "0.1uF" (at 60.96 255.27 90)
       (effects (font (size 1.27 1.27)) (justify left))
     )
@@
       (effects (font (size 1.27 1.27)) (justify left))
     )
-    (property "Footprint" "" (at 344.17 132.08 0)
+    (property "Footprint" "Resistor_SMD:R_0603_1608Metric" (at 344.17 132.08 0)
       (effects (font (size 1.27 1.27)) hide)
     )
@@
       (effects (font (size 1.27 1.27)) (justify left))
     )
-    (property "Footprint" "" (at 267.97 68.58 0)
+    (property "Footprint" "Resistor_SMD:R_0603_1608Metric" (at 267.97 68.58 0)
       (effects (font (size 1.27 1.27)) hide)
     )
@@
       (effects (font (size 1.27 1.27)) (justify left))
     )
-    (property "Value" "10uF" (at 311.15 196.85 0)
+    (property "Value" "0.1uF" (at 312.42 196.85 0)
       (effects (font (size 1.27 1.27)) (justify left))
     )
@@
       (effects (font (size 1.27 1.27)) (justify left))
     )
-    (property "Footprint" "" (at 256.54 57.15 0)
+    (property "Footprint" "Resistor_SMD:R_0603_1608Metric" (at 256.54 57.15 0)
       (effects (font (size 1.27 1.27)) hide)
     )
@@
       (effects (font (size 1.27 1.27)) (justify left))
     )
-    (property "Value" "10uF" (at 320.04 196.85 0)
+    (property "Value" "0.1uF" (at 320.04 196.85 0)
       (effects (font (size 1.27 1.27)) (justify left))
     )
@@
       (effects (font (size 1.27 1.27)) (justify left))
     )
-    (property "Footprint" "" (at 256.54 69.85 0)
+    (property "Footprint" "Resistor_SMD:R_0603_1608Metric" (at 256.54 69.85 0)
       (effects (font (size 1.27 1.27)) hide)
     )
@@
       (effects (font (size 1.27 1.27)) (justify left))
     )
-    (property "Value" "10uF" (at 293.37 196.85 0)
+    (property "Value" "0.1uF" (at 293.37 196.85 0)
       (effects (font (size 1.27 1.27)) (justify left))
     )
@@
       (effects (font (size 1.27 1.27)) (justify left))
     )
-    (property "Footprint" "" (at 261.62 146.05 0)
+    (property "Footprint" "Resistor_SMD:R_0603_1608Metric" (at 261.62 146.05 0)
       (effects (font (size 1.27 1.27)) hide)
     )
@@
       (effects (font (size 1.27 1.27)) (justify left))
     )
-    (property "Value" "10uF" (at 284.48 196.85 0)
+    (property "Value" "0.1uF" (at 284.48 196.85 0)
       (effects (font (size 1.27 1.27)) (justify left))
     )
@@
       (effects (font (size 1.27 1.27)) (justify left))
     )
-    (property "Footprint" "" (at 344.17 116.84 0)
+    (property "Footprint" "Resistor_SMD:R_0603_1608Metric" (at 344.17 116.84 0)
       (effects (font (size 1.27 1.27)) hide)
     )
@@
     )
   )
-  (symbol (lib_id "power:GND") (at 53.34 266.7 0) (unit 1)
+  (symbol (lib_id "power:GND") (at 53.34 265.43 0) (unit 1)
     (in_bom yes) (on_board yes) (dnp no) (fields_autoplaced)
-    (property "Reference" "#PWR014" (at 53.34 273.05 0)
+    (property "Reference" "#PWR014" (at 53.34 271.78 0)
       (effects (font (size 1.27 1.27)) hide)
     )
-    (property "Value" "GND" (at 53.34 271.78 0)
+    (property "Value" "GND" (at 53.34 270.51 0)
       (effects (font (size 1.27 1.27)))
     )
-    (property "Footprint" "" (at 53.34 266.7 0)
+    (property "Footprint" "" (at 53.34 265.43 0)
       (effects (font (size 1.27 1.27)) hide)
     )
-    (property "Datasheet" "" (at 53.34 266.7 0)
+    (property "Datasheet" "" (at 53.34 265.43 0)
       (effects (font (size 1.27 1.27)) hide)
     )
@@
       (effects (font (size 1.27 1.27)) (justify left))
     )
-    (property "Footprint" "" (at 350.52 39.37 0)
+    (property "Footprint" "Resistor_SMD:R_0603_1608Metric" (at 350.52 39.37 0)
       (effects (font (size 1.27 1.27)) hide)
     )
@@
       (effects (font (size 1.27 1.27)) (justify left))
     )
-    (property "Footprint" "" (at 308.61 60.96 0)
+    (property "Footprint" "Resistor_SMD:R_0603_1608Metric" (at 308.61 60.96 0)
       (effects (font (size 1.27 1.27)) hide)
     )
@@
       (effects (font (size 1.27 1.27)) (justify left))
     )
-    (property "Value" "10uF" (at 60.96 264.16 90)
+    (property "Value" "0.1uF" (at 60.96 264.16 90)
       (effects (font (size 1.27 1.27)) (justify left))
     )
@@
       (effects (font (size 1.27 1.27)) (justify left))
     )
-    (property "Footprint" "" (at 250.19 134.62 0)
+    (property "Footprint" "Resistor_SMD:R_0603_1608Metric" (at 250.19 134.62 0)
       (effects (font (size 1.27 1.27)) hide)
     )

Commit message: fixed GS_VBUS overtaking the GND symbol error, lesson learned, fixed PCB ratnest
Parts:
- removed BT1: TBD, symbol Device:Battery
- D1, D2: footprint PDS76013 -> sbr8u:POWERDI5
- IC1: footprint QFN40P400X400X80-33N-D -> bq2517:QFN40P400X400X80-33N-D
- IC2, IC3: footprint SOIC127P600X170-9N -> tps54:SOIC127P600X170-9N
- Q1, Q2, Q3, Q4: footprint CSD17308Q3 -> csd17:CSD17308Q3
- Q5: footprint DQG_VSON-CLIP -> csd25:DQG_VSON-CLIP
- R16: footprint (none) -> Resistor_SMD:R_0603_1608Metric
Connections:
- net GND: now also C12.1, C13.1, C14.1, C15.1, C16.1, C17.1; no longer C12.2, C13.2, C14.2, C15.2, C16.2, C17.2, C22.2, IC1.32 (SW1), L1.1, Q1.1 (S_1), Q1.2 (S_2), Q1.3 (S_3), Q2.5 (D_1), Q2.6 (D_2), Q2.7 (D_3), Q2.8 (D_4), Q2.9 (D_5), R12.2, R13.2, R15.1, R37.1
- net VBUS: now also C12.2, C13.2, C14.2, C15.2, C16.2, C17.2, R12.2, R13.2, R15.1, R37.1
- net BATT+: now reaches C31.1, R16.2, R18.1
- new net SW1: C22.2, IC1.32 (SW1), L1.1, Q1.1 (S_1), Q1.2 (S_2), Q1.3 (S_3), Q2.5 (D_1), Q2.6 (D_2), Q2.7 (D_3), Q2.8 (D_4), Q2.9 (D_5)
Other:
- moved on the sheet: R15

Commit message: some changes to schematic nets, grouping passives and mosfets around our charger ic in pcb editor
Changed lines of the file:
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@@
   (junction (at 59.69 248.92) (diameter 0) (color 0 0 0 0)
   )
+  (junction (at 149.86 114.3) (diameter 0) (color 0 0 0 0)
+  )
   (junction (at 261.62 222.25) (diameter 0) (color 0 0 0 0)
   )
@@
   (junction (at 218.44 213.36) (diameter 0) (color 0 0 0 0)
   )
+  (junction (at 149.86 118.11) (diameter 0) (color 0 0 0 0)
+  )
   (junction (at 186.69 213.36) (diameter 0) (color 0 0 0 0)
   )
@@
   (junction (at 59.69 213.36) (diameter 0) (color 0 0 0 0)
   )
-  (junction (at 140.97 114.3) (diameter 0) (color 0 0 0 0)
-  )
   (junction (at 80.01 143.51) (diameter 0) (color 0 0 0 0)
   )
@@
     (stroke (width 0) (type default))
   )
-  (wire (pts (xy 140.97 114.3) (xy 154.94 114.3))
-    (stroke (width 0) (type default))
-  )
   (wire (pts (xy 314.96 30.48) (xy 321.31 30.48))
     (stroke (width 0) (type default))
@@
     (stroke (width 0) (type default))
   )
-  (wire (pts (xy 138.43 114.3) (xy 140.97 114.3))
-    (stroke (width 0) (type default))
-  )
   (wire (pts (xy 60.96 83.82) (xy 60.96 86.36))
     (stroke (width 0) (type default))
@@
     (stroke (width 0) (type default))
   )
-  (wire (pts (xy 125.73 107.95) (xy 138.43 107.95))
-    (stroke (width 0) (type default))
-  )
   (wire (pts (xy 167.64 113.03) (xy 179.07 113.03))
     (stroke (width 0) (type default))
@@
     (stroke (width 0) (type default))
   )
+  (wire (pts (xy 138.43 107.95) (xy 125.73 107.95))
+    (stroke (width 0) (type default))
+  )
   (wire (pts (xy 67.31 123.19) (xy 80.01 123.19))
     (stroke (width 0) (type default))
@@
     (stroke (width 0) (type default))
   )
+  (wire (pts (xy 149.86 114.3) (xy 154.94 114.3))
+    (stroke (width 0) (type default))
+  )
   (wire (pts (xy 49.53 213.36) (xy 49.53 214.63))
     (stroke (width 0) (type default))
@@
     (stroke (width 0) (type default))
   )
-  (wire (pts (xy 138.43 107.95) (xy 138.43 114.3))
+  (wire (pts (xy 138.43 118.11) (xy 149.86 118.11))
+    (stroke (width 0) (type default))
+  )
+  (wire (pts (xy 138.43 107.95) (xy 138.43 118.11))
     (stroke (width 0) (type default))
   )
@@
     (stroke (width 0) (type default))
   )
-  (wire (pts (xy 140.97 115.57) (xy 140.97 114.3))
+  (wire (pts (xy 149.86 114.3) (xy 149.86 118.11))
     (stroke (width 0) (type default))
   )
@@
     (stroke (width 0) (type default))
   )
+  (wire (pts (xy 149.86 114.3) (xy 140.97 114.3))
+    (stroke (width 0) (type default))
+  )
   (wire (pts (xy 302.26 152.4) (xy 302.26 153.67))
     (stroke (width 0) (type default))
@@
     )
   )
-  (symbol (lib_id "power:GND") (at 140.97 115.57 0) (unit 1)
+  (symbol (lib_id "power:GND") (at 149.86 118.11 0) (unit 1)
     (in_bom yes) (on_board yes) (dnp no) (fields_autoplaced)
-    (property "Reference" "#PWR02" (at 140.97 121.92 0)
+    (property "Reference" "#PWR02" (at 149.86 124.46 0)
       (effects (font (size 1.27 1.27)) hide)
     )
-    (property "Value" "GND" (at 140.97 120.65 0)
+    (property "Value" "GND" (at 149.86 123.19 0)
       (effects (font (size 1.27 1.27)))
     )
-    (property "Footprint" "" (at 140.97 115.57 0)
+    (property "Footprint" "" (at 149.86 118.11 0)
       (effects (font (size 1.27 1.27)) hide)
     )
-    (property "Datasheet" "" (at 140.97 115.57 0)
+    (property "Datasheet" "" (at 149.86 118.11 0)
       (effects (font (size 1.27 1.27)) hide)
     )

Commit message: adding connectors for display and pi power, pin headers
Parts:
- removed C45: 0.1uF, Capacitor_SMD:C_0603_1608Metric, symbol Device:C_Small
- removed C46: 4700pf, Capacitor_SMD:C_0603_1608Metric, symbol Device:C_Small
- removed C47, C49: 100uF, Capacitor_SMD:C_0603_1608Metric, symbol Device:C_Small
- removed C48: 47pf, Capacitor_SMD:C_0603_1608Metric, symbol Device:C_Small
- removed D2: PDS760-13, sbr8u:POWERDI5, symbol psd760:PDS760-13
- removed IC3: TPS54540DDA, tps54:SOIC127P600X170-9N, symbol tps54:TPS54540DDA
- removed L3: 5.5uH, Inductor_SMD:L_0603_1608Metric, symbol Device:L
- removed R25: 365k, Resistor_SMD:R_0603_1608Metric, symbol Device:R_Small_US
- removed R26: 88.7k, Resistor_SMD:R_0603_1608Metric, symbol Device:R_Small_US
- removed R27: 243k, Resistor_SMD:R_0603_1608Metric, symbol Device:R_Small_US
- removed R28: 16.9k, Resistor_SMD:R_0603_1608Metric, symbol Device:R_Small_US
- removed R29: 31.6k, Resistor_SMD:R_0603_1608Metric, symbol Device:R_Small_US
- removed R30: 10.2k, Resistor_SMD:R_0603_1608Metric, symbol Device:R_Small_US
- added IC3, IC5: LP5907QMFX-3.0Q1, lp59:SOT95P280X145-5N, symbol lp59:LP5907QMFX-3.0Q1
- C41, C42, C43, C44: value 4.7uF -> 1uF
Connections:
- net VOUT1 is gone; now on net VOUT_5V: C37.2, C38.2, L2.2, R23.1
- net GND: now also IC3.2 (GND), IC5.2 (GND)
- net VOUT_5V: now reaches C41.2, C43.2
- net VOUT_5V: now also IC3.1 (IN), IC3.3 (EN), IC5.1 (IN), IC5.3 (EN); no longer C42.2, C44.2
- new net 3V3_MCU: C42.2, IC3.5 (OUT)
- new net 3V3_RADAR: C44.2, IC5.5 (OUT)

Commit message: changing sizes of caps from 06 to 04, also using vias on DW spi interfact to stm32
Parts:
- C1, C10, C12, C13, C14, C15, C16, C17, C18, C2, C22, C23, C24, C25, C26, C27, C28, C3, C30, C31, C4, C5, C8, C9: footprint Capacitor_SMD:C_0603_1608Metric -> Capacitor_SMD:C_0402_1005Metric
- R1, R10, R11, R16, R17, R18, R2, R3, R4, R5, R6, R9: footprint Resistor_SMD:R_0603_1608Metric -> Resistor_SMD:R_0402_1005Metric
Connections:
- net VSYS: now also C32.2, C33.2, C34.2, C35.2, IC2.2 (VIN), R20.1

Commit message: routing rails and BQ 4 switch mosfets
Changed lines of the file:
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@@
     )
     (property "Value" "4.99" (at 80.01 219.71 0)
-      (effects (font (size 1.27 1.27)) (justify right))
+      (effects (font (size 1.27 1.27)) (justify left))
     )
     (property "Footprint" "Resistor_SMD:R_0603_1608Metric" (at 86.36 218.44 0)
