File: pmics.kicad_sch (KiCad schematic)
At the start: 77 parts, among them IC1 BQ25713RSNR, IC2 TPS54540DDA, IC3 LP5907QMFX-3.0Q1, IC5 LP5907QMFX-3.0Q1, Q1 CSD17308Q3, Q2 CSD17308Q3, Q3 CSD17308Q3, Q4 CSD17308Q3, Q5 CSD25404Q3

Commit message: replacing battery charger inductor with the correct one capable of handling high current applications, updating user footprint lib. Doing some serious routing leaving the battery charger for last due to complexity
Parts:
- L1: footprint Inductor_SMD:L_0603_1608Metric -> induct:INDPM9785X300N
Connections:
- net GND: no longer Q4.5 (D_1), Q4.6 (D_2), Q4.7 (D_3), Q4.8 (D_4), Q4.9 (D_5), Q5.5 (S_1), Q5.6 (S_2), Q5.7 (S_3), Q5.8 (S_4)
- net VSYS: now also Q4.5 (D_1), Q4.6 (D_2), Q4.7 (D_3), Q4.8 (D_4), Q4.9 (D_5), Q5.5 (S_1), Q5.6 (S_2), Q5.7 (S_3), Q5.8 (S_4)
Other:
- moved on the sheet: L1
Changed lines of the file:
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@@
   (junction (at 125.73 243.84) (diameter 0) (color 0 0 0 0)
   )
+  (junction (at 269.24 191.77) (diameter 0) (color 0 0 0 0)
+  )
   (junction (at 161.29 248.92) (diameter 0) (color 0 0 0 0)
   )
@@
   (junction (at 87.63 226.06) (diameter 0) (color 0 0 0 0)
   )
-  (junction (at 269.24 199.39) (diameter 0) (color 0 0 0 0)
-  )
   (junction (at 57.15 123.19) (diameter 0) (color 0 0 0 0)
   )
@@
     (stroke (width 0) (type default))
   )
-  (wire (pts (xy 262.89 213.36) (xy 262.89 199.39))
+  (wire (pts (xy 262.89 191.77) (xy 262.89 213.36))
     (stroke (width 0) (type default))
   )
@@
     (stroke (width 0) (type default))
   )
-  (wire (pts (xy 198.12 213.36) (xy 203.2 213.36))
+  (wire (pts (xy 199.39 213.36) (xy 203.2 213.36))
     (stroke (width 0) (type default))
   )
@@
     (stroke (width 0) (type default))
   )
-  (wire (pts (xy 186.69 213.36) (xy 190.5 213.36))
+  (wire (pts (xy 186.69 213.36) (xy 191.77 213.36))
     (stroke (width 0) (type default))
   )
@@
     (stroke (width 0) (type default))
   )
-  (wire (pts (xy 262.89 199.39) (xy 269.24 199.39))
-    (stroke (width 0) (type default))
-  )
   (wire (pts (xy 226.06 213.36) (xy 236.22 213.36))
     (stroke (width 0) (type default))
@@
     (stroke (width 0) (type default))
   )
+  (wire (pts (xy 262.89 191.77) (xy 269.24 191.77))
+    (stroke (width 0) (type default))
+  )
   (wire (pts (xy 73.66 81.28) (xy 80.01 81.28))
     (stroke (width 0) (type default))
@@
     )
   )
-  (symbol (lib_id "Device:L") (at 194.31 213.36 90) (unit 1)
+  (symbol (lib_id "Device:L") (at 195.58 213.36 90) (unit 1)
     (in_bom yes) (on_board yes) (dnp no) (fields_autoplaced)
-    (property "Reference" "L1" (at 194.31 208.28 90)
+    (property "Reference" "L1" (at 195.58 208.28 90)
       (effects (font (size 1.27 1.27)))
     )
-    (property "Value" "2.2uH" (at 194.31 210.82 90)
+    (property "Value" "2.2uH" (at 195.58 210.82 90)
       (effects (font (size 1.27 1.27)))
     )
-    (property "Footprint" "Inductor_SMD:L_0603_1608Metric" (at 194.31 213.36 0)
+    (property "Footprint" "induct:INDPM9785X300N" (at 195.58 213.36 0)
       (effects (font (size 1.27 1.27)) hide)
     )
-    (property "Datasheet" "~" (at 194.31 213.36 0)
+    (property "Datasheet" "~" (at 195.58 213.36 0)
       (effects (font (size 1.27 1.27)) hide)
     )
@@
   )
   (symbol (lib_id "csd17:CSD17308Q3") (at 151.13 248.92 180) (unit 1)
-    (in_bom yes) (on_board yes) (dnp no) (fields_autoplaced)
+    (in_bom yes) (on_board yes) (dnp no)
     (property "Reference" "Q2" (at 138.43 231.14 0)
       (effects (font (size 1.27 1.27)))
@@
     (in_bom yes) (on_board yes) (dnp no)
     (property "Reference" "C18" (at 78.74 227.33 0)
-      (effects (font (size 1.27 1.27)) (justify left))
+      (effects (font (size 1.27 1.27)) (justify right))
     )
     (property "Value" "470nF" (at 80.01 229.87 0)

Commit message: replacing our indcutr for TPS with proper one, creating a bom tool for easier component selection and fitering, currently getting all my passives in order
Parts:
- C37, C38: footprint Capacitor_SMD:C_0603_1608Metric -> Capacitor_SMD:C_0805_2012Metric
- L2: footprint Inductor_SMD:L_0603_1608Metric -> 55induct:CDRH62BNP5R5NCB
Changed lines of the file:
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@@
       (effects (font (size 1.27 1.27)))
     )
-    (property "Footprint" "Inductor_SMD:L_0603_1608Metric" (at 311.15 30.48 0)
+    (property "Footprint" "55induct:CDRH62BNP5R5NCB" (at 311.15 30.48 0)
       (effects (font (size 1.27 1.27)) hide)
     )
@@
       (effects (font (size 1.27 1.27)) (justify left))
     )
-    (property "Footprint" "Capacitor_SMD:C_0603_1608Metric" (at 321.31 39.37 0)
+    (property "Footprint" "Capacitor_SMD:C_0805_2012Metric" (at 321.31 39.37 0)
       (effects (font (size 1.27 1.27)) hide)
     )
@@
       (effects (font (size 1.27 1.27)) (justify left))
     )
-    (property "Footprint" "Capacitor_SMD:C_0603_1608Metric" (at 332.74 39.37 0)
-      (effects (font (size 1.27 1.27)) hide)
-    )
+    (property "Footprint" "Capacitor_SMD:C_0805_2012Metric" (at 332.74 39.37 0)
+      (effects (font (size 1.27 1.27)) hide)
+    )
